Commit message: changed vito urdf to run dual manipolation

File: vito_description/robot/old_vito/vito_old.urdf.xacro (robot description, xacro)
@@ -7,30 +7,34 @@
   <xacro:include filename="$(find vito_description)/model/materials.urdf"/>
   <xacro:include filename="$(find lwr_description)/model/kuka_lwr.urdf.xacro"/>
-  <!-- <xacro:include filename="$(find soft_hand_description)/model/soft_hand_old.urdf.xacro"/> -->
   <xacro:include filename="$(find soft_hand_description)/model/soft_hand.urdf.xacro"/>
-  <xacro:include filename="$(find kit_head_description)/model/kit_head.urdf.xacro"/>
-  <link name="vito_anchor" />
+  <link name="world" />
+   <link name="vito_anchor"/>
+  <joint name="w_fixed" type="fixed">
+      <origin xyz="0.0 0.0 0.0" rpy="0 0 0"/>
+      <parent link="world" />
+      <child link="vito_anchor" />
+    </joint>
   <!-- BODY -->
-  <xacro:model_table name="table"
+<!--    <xacro:model_table name="table"
                     parent="vito_anchor"
                     length="0.725"
                     width="1.05"
                     height="0.910"
-                    plate_thickness="0.05">
-    <origin xyz="-0.495 0.55 0" rpy="0 0 0"/>
-  </xacro:model_table>
+		       plate_thickness="0.05">
+    <origin xyz="0.0 0.55 0" rpy="0 0 0"/>
+    </xacro:model_table> -->
   <!-- WORKBENCH -->
-  <xacro:model_table name="workbench"
-                    parent="vito_anchor"
-                    length="0.725"
-                    width="1.25"
-                    height="0.960"
-                    plate_thickness="0.1">
-  <origin xyz="-1.25 0.625 0.07" rpy="0 0 0"/>
-  </xacro:model_table>
+<!--   <xacro:model_table name="workbench" -->
+<!--                     parent="vito_anchor" -->
+<!--                     length="0.725" -->
+<!--                     width="1.25" -->
+<!--                     height="0.960" -->
+<!--                     plate_thickness="0.1"> -->
+<!--   <origin xyz="-1.25 0.625 0.07" rpy="0 0 0"/> -->
+<!--   </xacro:model_table> -->
   <!-- TORSO -->
-  <xacro:model_torso name="torso" parent="vito_anchor">
+   <xacro:model_torso name="torso" parent="vito_anchor"> -->
     <origin xyz="0 0 0"/>
-  </xacro:model_torso>
+   </xacro:model_torso>
   <!-- LEFT ARM -->
   <xacro:kuka_lwr name="left_arm" parent="vito_anchor">
@@ -43,13 +47,9 @@
   <!-- RIGHT ARM -->
   <xacro:kuka_lwr name="right_arm" parent="vito_anchor">
-    <origin xyz="-0.165 0.10858 0.390" rpy="-1.5707963267948966 0.5235987010713441 0.5235990737060282"/>
+    <origin xyz="-0.165 0.10858 0.390" rpy="-1.5707963267948966 -0.5235987010713441 0.5235990737060282"/>
   </xacro:kuka_lwr>
   <!-- RIGHT SOFTHAND -->
   <xacro:soft_hand parent="right_arm_7_link" name="right_hand" left="false" withAdaptiveTransmission="true" useMimicTag="$(arg use_mimic_tag)">
-    <origin xyz="0 0 0" rpy="0 0 0"/>
+    <origin xyz="0 0 0.0" rpy="0 0 0"/>
   </xacro:soft_hand>
-  <!-- HEAD -->
-  <xacro:kit_head name="head" parent="vito_anchor">
-    <origin xyz="0.0 0.0 ${0.55 + 0.1}" rpy="0.0 0.0 3.141592"/>
-  </xacro:kit_head>
 </robot>
