Commit message: fixed some visualization file and fixed display.launch for gazebo simulation

File: vito_description/model/velvet.urdf.xacro (robot description, xacro)
@@ -25,5 +25,5 @@
     <visual>
       <geometry>
-        <mesh filename="package://vito_description/meshes/gazebo_assieme.stl"/>
+        <mesh filename="package://vito_description/meshes/velvet_tray.stl"/>
       </geometry>
       <material name="Vito/Silver"/>
@@ -31,5 +31,5 @@
     <collision>
       <geometry>
-        <mesh filename="package://vito_description/meshes/gazebo_assieme.stl"/>
+        <mesh filename="package://vito_description/meshes/velvet_tray.stl"/>
       </geometry>
     </collision>

File: vito_description/robot/vito.urdf.xacro (robot description, xacro)
@@ -38,5 +38,5 @@
   </xacro:kuka_lwr>
   <!-- LEFT SOFTHAND -->
-  <xacro:soft_hand parent="left_arm_7_link" name="left_hand" left="true" withAdaptiveTransmission="true" useMimicTag="$(arg use_mimic_tag)">
+  <xacro:soft_hand parent="left_arm_7_link" name="left_hand" left="true" withAdaptiveTransmission="true" useMimicTag="true">
     <origin xyz="0 0 0" rpy="0 0 0"/>
   </xacro:soft_hand>
@@ -46,5 +46,5 @@
   </xacro:kuka_lwr>
   <!-- RIGHT SOFTHAND -->
-  <xacro:soft_hand parent="right_arm_7_link" name="right_hand" left="false" withAdaptiveTransmission="true" useMimicTag="$(arg use_mimic_tag)">
+  <xacro:soft_hand parent="right_arm_7_link" name="right_hand" left="false" withAdaptiveTransmission="true" useMimicTag="true">
     <origin xyz="0 0 0" rpy="0 0 0"/>
   </xacro:soft_hand>

File: vito_description/robot/vito_iliad.urdf.xacro (robot description, xacro)
@@ -98,5 +98,6 @@
    <xacro:model_velvet parent="left_arm_7_link" name="left_velvet">
     <!-- <origin xyz="0 0 0.14" rpy="0 0 0.5235987010713441"/>    -->
-    <origin xyz="0 0.07 0.121244" rpy="-0.5235987010713441 0 0"/>
+    <!-- <origin xyz="0 0.07 0.121244" rpy="-0.5235987010713441 0 0"/> -->
+    <origin xyz="0 0.035 0.151244" rpy="0 -0.5235987010713441 -1.57"/>
   </xacro:model_velvet>
 <link name="velvet_dummy">
