Commit message: changed vito-iliad urdf: fixed velvet orietation

File: vito_description/robot/vito_iliad.urdf.xacro (robot description, xacro)
@@ -90,7 +90,6 @@
 <!-- PALETTA LEFT -->
    <xacro:model_velvet parent="left_arm_7_link" name="left_velvet">
-    <origin xyz="0 0 0.14" rpy="0 0 0.5235987010713441"/>
-     <!-- <origin xyz="0 0 0.14" rpy="0 0 0"/>    -->
-    <!-- <origin xyz="0 0 0" rpy="0 0 0"/>    -->    <!-- conf inverse kinematic è pi ultima componente -->
+    <!-- <origin xyz="0 0 0.14" rpy="0 0 0.5235987010713441"/>    -->
+    <origin xyz="0 0 0.14" rpy="0 0 0"/>
   </xacro:model_velvet>
 <link name="velvet_dummy">

Commit message: fixed velvet orientation

File: vito_description/robot/vito_iliad.urdf.xacro (robot description, xacro)
@@ -89,7 +89,8 @@
   </joint>
 <!-- PALETTA LEFT -->
+<!-- the velvet tray has a 30° offset on the x axis wrt the 7th link -->
    <xacro:model_velvet parent="left_arm_7_link" name="left_velvet">
     <!-- <origin xyz="0 0 0.14" rpy="0 0 0.5235987010713441"/>    -->
-    <origin xyz="0 0 0.14" rpy="0 0 0"/>
+    <origin xyz="0 0.07 0.121244" rpy="-0.5235987010713441 0 0"/>
   </xacro:model_velvet>
 <link name="velvet_dummy">

Commit message: added ILIAD object meshes

File: vito_description/robot/vito_iliad.urdf.xacro (robot description, xacro)
@@ -9,6 +9,12 @@
   <xacro:include filename="$(find lwr_description)/model/kuka_lwr.urdf.xacro"/>
   <xacro:include filename="$(find soft_hand_description)/model/soft_hand.urdf.xacro"/>
+  <!-- show all the ILIAD objects TODO(ed): make this optional-->
+  <xacro:include filename="$(find vito_description)/robot/iliad_object_show.urdf.xacro"/>
   <link name="world" />
   <link name="vito_anchor" />
+    <!-- show all the ILIAD objects TODO(ed): make this optional-->
+    <xacro:iliad_object_show parent="world">
+      <origin xyz="0 0 0" rpy="0 0 0"/>
+    </xacro:iliad_object_show>
     <joint name="w_fixed" type="fixed">
       <origin xyz="0.0 0.0 0.0" rpy="0 0 0"/>

Commit message: added camera to robot model

File: vito_description/robot/vito_iliad.urdf.xacro (robot description, xacro)
@@ -2,4 +2,5 @@
 <robot xmlns:xacro="http://www.ros.org/wiki/xacro"
        name="vito">
+  <arg name="use_mimic_tag" default="false"/>
   <!-- MODELS -->
   <xacro:include filename="$(find vito_description)/model/torso.urdf.xacro"/>
@@ -9,55 +10,32 @@
   <xacro:include filename="$(find lwr_description)/model/kuka_lwr.urdf.xacro"/>
   <xacro:include filename="$(find soft_hand_description)/model/soft_hand.urdf.xacro"/>
+  <xacro:include filename="$(find youbot_description)/urdf/sensors/asus_xtion_camera.urdf.xacro"/>
   <!-- show all the ILIAD objects TODO(ed): make this optional-->
-  <xacro:include filename="$(find vito_description)/robot/iliad_object_show.urdf.xacro"/>
+  <!-- <xacro:include filename="$(find vito_description)/robot/iliad_object_show.urdf.xacro"/> -->
   <link name="world" />
   <link name="vito_anchor" />
+  <link name="camera_link"/>
+  <!-- <link name="camera_rgb_optical_frame"/> -->
     <!-- show all the ILIAD objects TODO(ed): make this optional-->
-    <xacro:iliad_object_show parent="world">
+    <!-- <xacro:iliad_object_show parent="world">
       <origin xyz="0 0 0" rpy="0 0 0"/>
-    </xacro:iliad_object_show>
+    </xacro:iliad_object_show> -->
     <joint name="w_fixed" type="fixed">
       <origin xyz="0.0 0.0 0.0" rpy="0 0 0"/>
-      <!-- <origin xyz="0.0 0.0 0.0" rpy="0 0 0"/> -->
       <parent link="world" />
       <child link="vito_anchor" />
     </joint>
-  <!-- BODY -->
- <!--  <xacro:model_table name="table"
-                    parent="world"
-                    length="0.725"
-                    width="1.05"
-                    height="0.910"
-                    plate_thickness="0.05">
-    <origin xyz="-0.215 0.55 0" rpy="0 0 0"/>
-  </xacro:model_table>
- -->
-    <!--xacro:model_table name="workbench"
-                    parent="world"
-                    length="0.725"
-                    width="1.25"
-                    height="0.910"
-                    plate_thickness="0.05">
-  <origin xyz="-1.25 0.625 0.00" rpy="0 0 0"/>
-  </xacro:model_table-->
-  <!-- TORSO -->
-  <!-- <xacro:model_torso name="torso" parent="world">
-    <origin xyz="0 0 0.0" rpy="0 0 0"/>
-  </xacro:model_torso> -->
+    <joint name="camera_kuka_base_joint" type="fixed">
+      <origin xyz="0.074 -0.087 0.088" rpy="-1.426 -1.539 -1.710"/>
+      <parent link="right_arm_7_link"/>
+      <child link="camera_link"/>
+    </joint>
   <!-- LEFT ARM -->
   <xacro:kuka_lwr name="left_arm" parent="vito_anchor">
-    <!-- <origin xyz="-0.1650   -0.0000    0.3814" rpy="-2.1588   -0.4478    1.8518"/> -->
     <origin xyz="0.57 0.801 1.307" rpy="3.1415 0.5235987010713441 3.1415"/>
-    <!-- <origin xyz="0.57 0.801 1.407" rpy="3.1415 0.5235987010713441 3.1415"/> -->        <!-- conf inverse kinematic -->
   </xacro:kuka_lwr>
-  <!-- LEFT SOFTHAND -->
- <!--  <xacro:soft_hand parent="left_arm_7_link" name="left_hand" left="true" withAdaptiveTransmission="true" useMimicTag="$(arg use_mimic_tag)">
-    <origin xyz="0 0 0" rpy="0 0 0"/>
-  </xacro:soft_hand> -->
   <!-- RIGHT ARM -->
-    <xacro:kuka_lwr name="right_arm" parent="vito_anchor">
-    <!-- <origin xyz="-0.165 0.10858 0.490" rpy="-1.5707963267948966 -0.5235987010713441 0.5235990737060282"/> -->
-     <origin xyz="0.77 0.801 1.607" rpy="3.1415 -0.7854 0"/>
- <!--  <origin xyz="0.77 0.801 1.707" rpy="3.1415 -0.7854 0"/> -->      <!-- conf originale inverse kinematic -->
+  <xacro:kuka_lwr name="right_arm" parent="vito_anchor">
+    <origin xyz="0.77 0.801 1.607" rpy="3.1415 -0.7854 0"/>
   </xacro:kuka_lwr>
   <!-- RIGHT SOFTHAND -->
@@ -66,26 +44,15 @@
   </xacro:soft_hand>
   <link name="ft_surface">
-      <inertial>
-        <mass value="0.1"/>
-          <origin xyz="0 0 0.0" rpy="0 0 0"/>
-            <inertia ixx="${1 / 12  * (3 * 0.05 * 0.05 + 0.01 * 0.01)}"  ixy="0"  ixz="0" iyy="${1 / 12  * (3 * 0.05 * 0.05 + 0.01 * 0.01)}" iyz="0" izz="${1 / 12  * (3 * 0.05 * 0.05 + 0.01 * 0.01)}" />
-      </inertial>
-      <visual>
-        <origin xyz="0 0 0.0" rpy="0 0 0"/>
-        <geometry>
-          <sphere radius="0.001" />
-        </geometry>
-      </visual>
-<!--       <collision>
-        <origin xyz="0 0 0.0" rpy="0 0 0"/>
-        <geometry>
-          <sphere radius="0.02" />
-        </geometry>
-        <surface>
-          <contact>
-            <collide_bitmask>"0x11111"</collide_bitmask>
-          </contact>
-        </surface>
-      </collision> -->
+    <inertial>
+      <mass value="0.1"/>
+      <origin xyz="0 0 0.0" rpy="0 0 0"/>
+      <inertia ixx="${1 / 12  * (3 * 0.05 * 0.05 + 0.01 * 0.01)}"  ixy="0"  ixz="0" iyy="${1 / 12  * (3 * 0.05 * 0.05 + 0.01 * 0.01)}" iyz="0" izz="${1 / 12  * (3 * 0.05 * 0.05 + 0.01 * 0.01)}" />
+    </inertial>
+    <visual>
+      <origin xyz="0 0 0.0" rpy="0 0 0"/>
+      <geometry>
+        <sphere radius="0.001" />
+      </geometry>
+    </visual>
   </link>
   <joint name="ft_joint_sensor" type="fixed">
@@ -94,77 +61,36 @@
     <child link="ft_surface" />
   </joint>
-<!-- PALETTA LEFT -->
+<!-- VELVET LEFT -->
 <!-- the velvet tray has a 30° offset on the x axis wrt the 7th link -->
-   <xacro:model_velvet parent="left_arm_7_link" name="left_velvet">
-    <!-- <origin xyz="0 0 0.14" rpy="0 0 0.5235987010713441"/>    -->
-    <!-- <origin xyz="0 0.07 0.121244" rpy="-0.5235987010713441 0 0"/> -->
+  <xacro:model_velvet parent="left_arm_7_link" name="left_velvet">
     <origin xyz="0 0.035 0.151244" rpy="0 -0.5235987010713441 -1.57"/>
   </xacro:model_velvet>
-<link name="velvet_dummy">
-</link>
-<joint name="velvet_dummy_joint" type="fixed">
-      <origin xyz="0.0150 -0.0260 0.28" rpy="0 0 0.5235987010713441"/>
-      <parent link="left_arm_7_link"/>
-      <child link="velvet_dummy"/>
-    </joint>
-<link name="hand_dummy">
-</link>
-<joint name="hand_dummy_joint" type="fixed">
-      <origin xyz="0 0 0.2" rpy="0 0 0"/>
-      <parent link="right_arm_7_link"/>
-      <child link="hand_dummy"/>
-    </joint>
-<!--
-  <link name="gripper_link">
-      <inertial>
-        <mass value="0.1"/>
-          <origin xyz="0 0 0.0" rpy="0 0 0"/>
-            <inertia ixx="${1 / 12  * (3 * 0.05 * 0.05 + 0.01 * 0.01)}"  ixy="0"  ixz="0" iyy="${1 / 12  * (3 * 0.05 * 0.05 + 0.01 * 0.01)}" iyz="0" izz="${1 / 12  * (3 * 0.05 * 0.05 + 0.01 * 0.01)}" />
-      </inertial>
-      <visual>
-        <origin xyz="0 0 0.0" rpy="0 0 0"/>
-        <geometry>
-        <mesh filename="package://vito_description/meshes/gripper.stl"/>
-        </geometry>
-      </visual>
-      <collision>
-        <origin xyz="0 0 0.0" rpy="0 0 0"/>
-        <geometry>
-          <sphere radius="0.02" />
-        </geometry>
-        <surface>
-          <contact>
-            <collide_bitmask>"0x11111"</collide_bitmask>
-          </contact>
-        </surface>
-      </collision>
+  <link name="velvet_dummy">
   </link>
-  <joint name="gripper_joint" type="fixed">
-    <origin xyz="0 0 0" rpy="0 0 0"/>
-    <parent link="left_arm_7_link" />
-    <child link="gripper_link" />
+  <joint name="velvet_dummy_joint" type="fixed">
+    <origin xyz="0.0150 -0.0260 0.28" rpy="0 0 0.5235987010713441"/>
+    <parent link="left_arm_7_link"/>
+    <child link="velvet_dummy"/>
   </joint>
- -->
-<!--   <gazebo reference="ft_surface_fake">
-    <gravity>true</gravity>
-  </gazebo>
-    <gazebo>
-      <plugin name="force_sensor" filename="libgazebo_ros_ft_sensor.so">
-        <updateRate>100.0</updateRate>
-        <topicName>ft_sensor_topic</topicName>
-        <jointName>ft_joint_sensor</jointName>
-      </plugin>
-    </gazebo>
-    <gazebo reference="ft_joint_sensor">
-      <provideFeedback>true</provideFeedback>
-      <disableFixedJointLumping>true</disableFixedJointLumping>
-    </gazebo>  -->
-    <xacro:model_table name="table"
-                    parent="world"
-                    length="0.6"
-                    width="0.8"
-                    height="0.70"
-                    plate_thickness="0.05">
+  <link name="hand_dummy">
+  </link>
+  <joint name="hand_dummy_joint" type="fixed">
+    <origin xyz="0 0 0.2" rpy="0 0 0"/>
+    <parent link="right_arm_7_link"/>
+    <child link="hand_dummy"/>
+  </joint>
+  <!-- CAMERA -->
+  <xacro:asus_xtion_camera name="camera_rviz" parent="camera_link" tilt="0">
+    <!-- <origin xyz="0.01 0.037 0" rpy="1.5708 -1.5708 0"/> -->
+    <origin xyz="-0.05 -0.10 -0.03" rpy="0 0 0"/>
+  </xacro:asus_xtion_camera>
+  <!-- ENVIRONMENT -->
+  <xacro:model_table name="table"
+                     parent="world"
+                     length="0.6"
+                     width="0.8"
+                     height="0.70"
+                     plate_thickness="0.05">
     <origin xyz="1.350 1.201 0.70" rpy="0 0 0"/>
-</xacro:model_table>
+  </xacro:model_table>
 </robot>

Commit message: iliad updated to floating base, no more fixed base

File: vito_description/robot/vito_iliad.urdf.xacro (robot description, xacro)
@@ -13,22 +13,63 @@
   <!-- show all the ILIAD objects TODO(ed): make this optional-->
   <!-- <xacro:include filename="$(find vito_description)/robot/iliad_object_show.urdf.xacro"/> -->
+  <!-- show all the ILIAD objects TODO(ed): make this optional-->
+  <!-- <xacro:iliad_object_show parent="world">
+    <origin xyz="0 0 0" rpy="0 0 0"/>
+  </xacro:iliad_object_show> -->
   <link name="world" />
   <link name="vito_anchor" />
   <link name="camera_link"/>
-  <!-- <link name="camera_rgb_optical_frame"/> -->
-    <!-- show all the ILIAD objects TODO(ed): make this optional-->
-    <!-- <xacro:iliad_object_show parent="world">
-      <origin xyz="0 0 0" rpy="0 0 0"/>
-    </xacro:iliad_object_show> -->
-    <joint name="w_fixed" type="fixed">
-      <origin xyz="0.0 0.0 0.0" rpy="0 0 0"/>
-      <parent link="world" />
-      <child link="vito_anchor" />
-    </joint>
-    <joint name="camera_kuka_base_joint" type="fixed">
-      <origin xyz="0.074 -0.087 0.088" rpy="-1.426 -1.539 -1.710"/>
-      <parent link="right_arm_7_link"/>
-      <child link="camera_link"/>
-    </joint>
+  <!-- ENVIRONMENT -->
+  <xacro:model_table name="table"
+                     parent="world"
+                     length="0.6"
+                     width="0.8"
+                     height="0.70"
+                     plate_thickness="0.05">
+    <origin xyz="1.350 1.201 0.70" rpy="0 0 0"/>
+  </xacro:model_table>
+  <!-- ROBOT -->
+  <!-- floating base for the robot, chain of x-y-z-yaw joints (floating does not work) -->
+  <link name="world_1" />
+  <link name="world_2" />
+  <link name="world_3" />
+  <joint name="world_x" type="prismatic">
+    <origin xyz="0.0 0.0 0.0" rpy="0 0 0"/>
+    <limit effort="1000.0" lower="-1000" upper="10000" velocity="10000"/>
+    <axis xyz="1 0 0"/>
+    <parent link="world" />
+    <child link="world_1" />
+  </joint>
+  <joint name="world_y" type="prismatic">
+    <origin xyz="0.0 0.0 0.0" rpy="0 0 0"/>
+    <limit effort="1000.0" lower="-1000" upper="10000" velocity="10000"/>
+    <axis xyz="0 1 0"/>
+    <parent link="world_1" />
+    <child link="world_2" />
+  </joint>
+  <joint name="world_z" type="prismatic">
+    <origin xyz="0.0 0.0 0.0" rpy="0 0 0"/>
+    <limit effort="1000.0" lower="-1000" upper="10000" velocity="10000"/>
+    <axis xyz="0 0 1"/>
+    <parent link="world_2" />
+    <child link="world_3" />
+  </joint>
+  <joint name="world_yaw" type="revolute">
+    <origin xyz="0.0 0.0 0.0" rpy="0 0 0"/>
+    <limit effort="1000.0" lower="-1000" upper="10000" velocity="10000"/>
+    <axis xyz="0 0 1"/>
+    <parent link="world_3" />
+    <child link="vito_anchor" />
+  </joint>
+  <!-- floating base for the robot END -->
+  <joint name="camera_kuka_base_joint" type="fixed">
+    <origin xyz="0.074 -0.087 0.088" rpy="-1.426 -1.539 -1.710"/>
+    <parent link="right_arm_7_link"/>
+    <child link="camera_link"/>
+  </joint>
+  <!-- CAMERA -->
+  <xacro:asus_xtion_camera name="camera_rviz" parent="camera_link" tilt="0">
+    <origin xyz="-0.05 -0.10 -0.03" rpy="0 0 0"/>
+  </xacro:asus_xtion_camera>
   <!-- LEFT ARM -->
   <xacro:kuka_lwr name="left_arm" parent="vito_anchor">
@@ -80,17 +121,3 @@
     <child link="hand_dummy"/>
   </joint>
-  <!-- CAMERA -->
-  <xacro:asus_xtion_camera name="camera_rviz" parent="camera_link" tilt="0">
-    <!-- <origin xyz="0.01 0.037 0" rpy="1.5708 -1.5708 0"/> -->
-    <origin xyz="-0.05 -0.10 -0.03" rpy="0 0 0"/>
-  </xacro:asus_xtion_camera>
-  <!-- ENVIRONMENT -->
-  <xacro:model_table name="table"
-                     parent="world"
-                     length="0.6"
-                     width="0.8"
-                     height="0.70"
-                     plate_thickness="0.05">
-    <origin xyz="1.350 1.201 0.70" rpy="0 0 0"/>
-  </xacro:model_table>
 </robot>
